File: zener-rng/zener-rng.sch (KiCad schematic (older format))
At the start: 51 parts

Commit message: Finish first schematic iteration
Parts:
- removed C?: 10uF, agg:0603, symbol agg-kicad:C
- removed C?: 1.5uF, agg:1206, symbol agg-kicad:C
- removed IC?: MCP1700T-5002E/TT, agg:SOT-23, symbol agg-kicad:MCP1700
- removed J?: CONN_01x03, symbol agg-kicad:CONN_01x03
- removed R?: 1k, agg:0603, symbol agg-kicad:R
- removed R?: 3k, agg:0603, symbol agg-kicad:R
- removed R?: 4.7k, agg:0603, symbol agg-kicad:R
- removed U?: TPL0401A-10QDCKRQ1, agg:SC-70-6, symbol TPL0401A-10QDCKRQ1:TPL0401A-10QDCKRQ1
- added IC1: MCP1700, agg:SOT-23, symbol agg-kicad:MCP1700
- added J2, J4: CONN_01x03, agg:SIL-254P-03, symbol agg-kicad:CONN_01x03
- added R15: 4.7k, agg:0603, symbol agg-kicad:R
- added TP11, TP12, TP13, TP14: TESTPAD, agg:TESTPAD, symbol agg-kicad:TESTPAD
- added U3: TPL0401A-10QDCKRQ1, agg:SC-70-6, symbol TPL0401A-10QDCKRQ1:TPL0401A-10QDCKRQ1
- added X1: Jumper, symbol agg-kicad:PART
- J3: renamed from J?; footprint (none) -> agg:SIL-254P-03; Farnell (none) -> 9731083
- J5: renamed from J?; footprint (none) -> agg:SIL-254P-03; Farnell (none) -> 1593459
- R12: renamed from R?; footprint (none) -> zener-rng:3266W_trimpot; Farnell (none) -> 9352651
- gave numbers to parts that had none: 40
Connections:
- net labels added: 3v3, VCC
- net labels removed: 5v
- wire segments 120 -> 149
- no-connect marks 6 -> 5
Other:
- note added: "Adjustable Reference"
- note added: "Alternative power input"
- note added: "Electronic control"
- note added: "Gnd"
- note added: "Manual control"
- note added: "Noise Generator"
- note added: "Noise out"
- note added: "Power"
- note added: "Power flag for KiCad"
- note added: "Ref out"
- note added: "SCL"
- note added: "SDA"
- note added: "Use jumper to select either manual or \nelectronic control of reference voltage"
- note removed: "- Noise out\n- i2c clk\n- i2c data\n- gnd\n- 3x pot jumper\n- bias out"
- note removed: "Use up these resistors\n(usually sold in 10s)"

Commit message: Begin PCB
Parts:
- added C11: 100nF, agg:0603, symbol agg-kicad:C
- C9: value 10nF -> 100nF; Farnell 1327675 -> 2749806
Connections:
- wire segments 149 -> 155
Changed lines of the file:
@@
 P 5150 5150
 F 0 "C9" V 5154 5208 50  0000 L CNN
-F 1 "10nF" V 5245 5208 50  0000 L CNN
+F 1 "100nF" V 5245 5208 50  0000 L CNN
 F 2 "agg:0603" H 5150 5150 50  0001 C CNN
 F 3 "" H 5150 5150 50  0001 C CNN
-F 4 "1327675" H 5150 5150 50  0001 C CNN "Farnell"
+F 4 "2749806" H 5150 5150 50  0001 C CNN "Farnell"
 	1    5150 5150
 	0    1    1    0
@@
 Connection ~ 2350 850
 $Comp
-L ST8R00:ST8R00 U1
-U 1 1 5C854A76
-P 2900 2500
-F 0 "U1" H 2410 2546 50  0000 R CNN
-F 1 "ST8R00" H 2410 2455 50  0000 R CNN
-F 2 "zener-rng:DFN-8-ST" V 2750 2000 50  0001 C CNN
-F 3 "http://www.farnell.com/datasheets/2581721.pdf" V 2750 2000 50  0001 C CNN
-F 4 "2849799" H 3100 2650 50  0001 C CNN "Farnell"
-	1    2900 2500
-	1    0    0    -1
-$EndComp
-$Comp
-L agg-kicad:GND #PWR0113
-U 1 1 5C854C66
-P 2750 3150
-F 0 "#PWR0113" H 2620 3190 50  0001 L CNN
-F 1 "GND" H 2850 3100 50  0000 C CNN
-F 2 "" H 2750 3150 50  0001 C CNN
-F 3 "" H 2750 3150 50  0001 C CNN
-	1    2750 3150
-	-1   0    0    -1
-$EndComp
-$Comp
 L agg-kicad:GND #PWR0114
 U 1 1 5C856299
-P 2850 3150
-F 0 "#PWR0114" H 2720 3190 50  0001 L CNN
+P 2900 3200
+F 0 "#PWR0114" H 2770 3240 50  0001 L CNN
 F 1 "GND" H 2900 3050 50  0000 C CNN
-F 2 "" H 2850 3150 50  0001 C CNN
-F 3 "" H 2850 3150 50  0001 C CNN
-	1    2850 3150
-	1    0    0    -1
-$EndComp
-$Comp
-L agg-kicad:GND #PWR0115
-U 1 1 5C8562F5
-P 3050 3150
-F 0 "#PWR0115" H 2920 3190 50  0001 L CNN
-F 1 "GND" H 3150 3100 50  0000 C CNN
-F 2 "" H 3050 3150 50  0001 C CNN
-F 3 "" H 3050 3150 50  0001 C CNN
-	1    3050 3150
+F 2 "" H 2900 3200 50  0001 C CNN
+F 3 "" H 2900 3200 50  0001 C CNN
+	1    2900 3200
 	1    0    0    -1
 $EndComp
@@
 P 8050 1850
 F 0 "#PWR0125" H 7920 1890 50  0001 L CNN
-F 1 "GND" H 7950 1850 50  0000 C CNN
+F 1 "GND" H 8150 1850 50  0000 C CNN
 F 2 "" H 8050 1850 50  0001 C CNN
 F 3 "" H 8050 1850 50  0001 C CNN
@@
 $EndComp
 $Comp
-L agg-kicad:GND #PWR?
+L agg-kicad:GND #PWR0136
 U 1 1 5CA04F12
 P 750 1800
-F 0 "#PWR?" H 620 1840 50  0001 L CNN
+F 0 "#PWR0136" H 620 1840 50  0001 L CNN
 F 1 "GND" H 750 1700 50  0000 C CNN
 F 2 "" H 750 1800 50  0001 C CNN
@@
 Text Notes 800  1800 0    50   ~ 0
 Power flag for KiCad
+$Comp
+L ST8R00:ST8R00 U1
+U 1 1 5CA16A54
+P 2900 2500
+F 0 "U1" H 2410 2546 50  0000 R CNN
+F 1 "ST8R00" H 2410 2455 50  0000 R CNN
+F 2 "zener-rng:DFN-8-ST" H 2900 1350 50  0001 C CNN
+F 3 "http://www.farnell.com/datasheets/2581721.pdf" H 2900 1450 50  0001 C CNN
+F 4 "2849799" H 2900 1250 50  0001 C CNN "Farnell"
+	1    2900 2500
+	1    0    0    -1
+$EndComp
+Wire Wire Line
+	2750 3150 2850 3150
+Connection ~ 2850 3150
+Wire Wire Line
+	2850 3150 2900 3150
+Wire Wire Line
+	2950 3100 2950 3150
+Connection ~ 2950 3150
+Wire Wire Line
+	2950 3150 3050 3150
+Wire Wire Line
+	2900 3200 2900 3150
+Connection ~ 2900 3150
+Wire Wire Line
+	2900 3150 2950 3150
+$Comp
+L agg-kicad:C C11
+U 1 1 5CA29BE8
+P 8050 1700
+F 0 "C11" V 8054 1758 50  0000 L CNN
+F 1 "100nF" V 8145 1758 50  0000 L CNN
+F 2 "agg:0603" H 8050 1700 50  0001 C CNN
+F 3 "" H 8050 1700 50  0001 C CNN
+F 4 "2749806" H 8050 1700 50  0001 C CNN "Farnell"
+	1    8050 1700
+	0    1    1    0
+$EndComp
+Connection ~ 8050 1700
+Connection ~ 8050 1800
 $EndSCHEMATC

Commit message: More work on PCB
Connections:
- net labels added: SCL, SDA
- wire segments 155 -> 153
- no-connect marks 5 -> 7
Other:
- note added: "flip"
- note removed: "SCL"
- note removed: "SDA"
Changed lines of the file:
@@
 L agg-kicad:CONN_01x03 J5
 U 1 1 5C88716D
-P 9650 2200
-F 0 "J5" H 9650 1850 50  0000 R CNN
-F 1 "CONN_01x03" H 9650 2300 50  0000 R CNN
-F 2 "agg:SIL-254P-03" H 9650 2200 50  0001 C CNN
-F 3 "" H 9650 2200 50  0001 C CNN
-F 4 "1593459" H 9650 2200 50  0001 C CNN "Farnell"
-	1    9650 2200
-	-1   0    0    1
+P 10100 1900
+F 0 "J5" H 10100 1550 50  0000 R CNN
+F 1 "CONN_01x03" H 10100 2000 50  0000 R CNN
+F 2 "agg:SIL-254P-03" H 10100 1900 50  0001 C CNN
+F 3 "" H 10100 1900 50  0001 C CNN
+F 4 "1593459" H 10100 1900 50  0001 C CNN "Farnell"
+	1    10100 1900
+	-1   0    0    -1
 $EndComp
 $Comp
@@
 $EndComp
 $Comp
-L agg-kicad:GND #PWR0131
-U 1 1 5C92F5CE
-P 9500 2250
-F 0 "#PWR0131" H 9370 2290 50  0001 L CNN
-F 1 "GND" H 9400 2250 50  0000 C CNN
-F 2 "" H 9500 2250 50  0001 C CNN
-F 3 "" H 9500 2250 50  0001 C CNN
-	1    9500 2250
-	1    0    0    -1
-$EndComp
-Wire Wire Line
-	9550 2200 9500 2200
-Wire Wire Line
-	9500 2200 9500 2250
-$Comp
 L agg-kicad:PART X1
 U 1 1 5C933AB8
@@
 Wire Wire Line
 	1400 800  1400 850
-Wire Wire Line
-	1450 1150 1200 1150
-Wire Wire Line
-	1200 1150 1200 1250
 Connection ~ 1200 1250
 Wire Wire Line
 	1450 1050 1200 1050
-Wire Wire Line
-	1200 1050 1200 1150
-Connection ~ 1200 1150
 $Comp
 L agg-kicad:3v3 #PWR0133
@@
 Text Notes 7000 5550 0    50   ~ 0
 Gnd
-Text Notes 9750 2200 0    50   ~ 0
-Gnd
-Text Notes 9750 2000 0    50   ~ 0
-SCL
-Text Notes 9750 2100 0    50   ~ 0
-SDA
 Text Notes 6200 2050 1    50   ~ 0
 Manual control
@@
 Wire Wire Line
 	9050 1950 9050 2000
-Connection ~ 9050 2000
-Wire Wire Line
-	9050 2000 9550 2000
 Wire Wire Line
 	9050 2150 9050 2100
-Connection ~ 9050 2100
-Wire Wire Line
-	9050 2100 9550 2100
 $Comp
 L agg-kicad:PWR #FLG0101
@@
 Connection ~ 8050 1700
 Connection ~ 8050 1800
+NoConn ~ 10000 1900
+Wire Wire Line
+	1200 1050 1200 1250
+NoConn ~ 1450 1150
+Text Label 9800 2000 0    50   ~ 0
+SDA
+Text Label 9800 2100 0    50   ~ 0
+SCL
+Text Label 9550 2000 2    50   ~ 0
+SCL
+Text Label 9550 2100 2    50   ~ 0
+SDA
+Wire Wire Line
+	9550 2000 9050 2000
+Connection ~ 9050 2000
+Wire Wire Line
+	9550 2100 9050 2100
+Connection ~ 9050 2100
+Text Notes 9600 2050 0    50   ~ 0
+flip
+Wire Wire Line
+	9800 2000 10000 2000
+Wire Wire Line
+	9800 2100 10000 2100
 $EndSCHEMATC

Commit message: Remove digital potentiometer from project
Parts:
- removed C11: 100nF, agg:0603, symbol agg-kicad:C
- removed J3, J5: CONN_01x03, agg:SIL-254P-03, symbol agg-kicad:CONN_01x03
- removed R15: 4.7k, agg:0603, symbol agg-kicad:R
- removed TP12, TP13, TP14: TESTPAD, agg:TESTPAD, symbol agg-kicad:TESTPAD
- removed U3: TPL0401A-10QDCKRQ1, agg:SC-70-6, symbol TPL0401A-10QDCKRQ1:TPL0401A-10QDCKRQ1
- removed X1: Jumper, symbol agg-kicad:PART
- added R14: 2.49k, agg:0603, symbol agg-kicad:R
- R15: renamed from R12; value potentiometer -> 1k potentiometer; Farnell 9352651 -> 9352643
- R16: value 4.7k -> 2.49k; Farnell 1652884 -> 1469767
- renumbered C4 to C2, C2 to C3, C3 to C4, C8 to C6, C6 to C7, C7 to C8, J4 to J3, R13 to R12, R14 to R13, R8 to R6, R9 to R7, R6 to R8, R7 to R9, TP3 to TP2, TP2 to TP3
Connections:
- net labels removed: SCL, SDA
- wire segments 153 -> 131
- no-connect marks 7 -> 6
Other:
- note added: "Use 2.49k resistors to reduce\ntrimmer wiper range\n(since we aim to keep within\nthe comparator's common\nmode region)"
- note removed: "Adjustable Reference"
- note removed: "Electronic control"
- note removed: "Manual control"
- note removed: "Use jumper to select either manual or \nelectronic control of reference voltage"
- note removed: "flip"

Commit message: Finish first revision of PCB
Parts:
- C4, C8: Farnell 2611923RL -> 2611923
Changed lines of the file:
@@
 F 2 "agg:0603" H 3800 2550 50  0001 C CNN
 F 3 "" H 3800 2550 50  0001 C CNN
-F 4 "2611923RL" H 3800 2550 50  0001 C CNN "Farnell"
+F 4 "2611923" H 3800 2550 50  0001 C CNN "Farnell"
 	1    3800 2550
 	0    1    -1   0
@@
 F 2 "agg:0603" H 2600 1950 50  0001 C CNN
 F 3 "" H 2600 1950 50  0001 C CNN
-F 4 "2611923RL" H 2600 1950 50  0001 C CNN "Farnell"
+F 4 "2611923" H 2600 1950 50  0001 C CNN "Farnell"
 	1    2600 1950
 	0    1    -1   0
