File: zener-rng/zener-rng.kicad_pcb (KiCad board)
At the start: 2 copper layers, 42 x 36 mm, 53 parts, among them IC1 MCP1700, J1 MICROUSB, J2 CONN_01x03, J3 CONN_01x03, J4 CONN_01x03, J5 CONN_01x03, Q1 2N4401, U1 ST8R00, U2 LT1215CS8#PBF, U3 TPL0401A-10QDCKRQ1

Commit message: More work on PCB
Parts:
- moved TP13 6.50 mm to (113.0, 127.0)
- moved TP14 6.50 mm to (113.0, 120.5)
- moved R7 4.96 mm to (87.8, 133.4), turned to 90 degrees
- moved C5 3.72 mm to (94.8, 144.5), turned to 270 degrees
- moved J5 2.50 mm to (120.0, 122.5), turned to 270 degrees
- moved R15 2.50 mm to (112.0, 125.0)
- moved R16 2.50 mm to (112.0, 122.5)
- moved TP6 1.77 mm to (87.8, 136.2)
- moved C6 1.00 mm to (100.0, 128.5), turned to 270 degrees
- moved TP4 0.79 mm to (96.2, 148.8)
- moved C10 0.75 mm to (110.2, 143.0)
- moved C3 0.75 mm to (87.8, 130.0)
- moved C7 0.75 mm to (96.2, 130.5)
- moved C8 0.75 mm to (114.0, 148.0)
- moved R10 0.75 mm to (110.2, 148.0)
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Connections:
- net Net-(J5-Pad2) renamed /SDA
- net Net-(J5-Pad3) renamed /SCL
- J2 pad 1: GND -> Net-(J2-Pad1)
- J5 pad 1: GND -> Net-(J5-Pad1)
Routing:
- net VCC: track 0.00 -> 61.3 mm
- net 12v: track 0.00 -> 49.3 mm
- net Net-(C4-Pad2): track 0.00 -> 20.6 mm
- net GND: track 0.00 -> 18.8 mm, vias 0 -> 12
- net Net-(R8-Pad2): track 0.00 -> 16.5 mm
- net 3v3: track 0.00 -> 14.4 mm
- net Net-(J3-Pad3): track 0.00 -> 11.4 mm
- net Net-(C10-Pad1): track 0.00 -> 10.1 mm
- net Net-(C4-Pad1): track 0.00 -> 9.52 mm
- net Net-(R6-Pad2): track 0.00 -> 8.86 mm
- net Net-(C10-Pad2): track 0.00 -> 8.34 mm
- net Net-(D1-Pad1): track 0.00 -> 7.29 mm
- net Net-(R8-Pad1): track 0.00 -> 6.93 mm
- net Net-(R10-Pad1): track 0.00 -> 6.26 mm
- net Net-(J3-Pad1): track 0.00 -> 6.18 mm
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- added copper zone on B.Cu, net GND
Other:
- board text added: "1.22V"
- board text added: "TP1"
- board text removed: "1.22V TPXX"

Commit message: Remove digital potentiometer from project
Parts:
- removed C11: 100nF, agg:0603
- removed J4, J5: CONN_01x03, agg:SIL-254P-03
- removed TP12, TP13, TP14: TESTPAD, agg:TESTPAD
- removed U3: TPL0401A-10QDCKRQ1, agg:SC-70-6
- C2: value 1.5uF -> 4.7nF; footprint agg:1206 -> agg:0603
- C3, C7: value 10uF -> 1.5uF; footprint agg:0603 -> agg:1206
- C4: value 4.7nF -> 10uF
- C6: value 1.5uF -> 33nF; footprint agg:1206 -> agg:0603
- C8: value 33nF -> 10uF
- R12: value potentiometer -> 1k; footprint zener-rng:3266W_trimpot -> agg:0603
- R14: value 1k -> 2.49k
- R15: value 4.7k -> 1k potentiometer; footprint agg:0603 -> zener-rng:3266W_trimpot
- R16: value 4.7k -> 2.49k
- R6: value 180k -> 2.49k
- R7: value 20k -> 249
- R8: value 2.49k -> 180k
- R9: value 249 -> 20k
- moved C8 28.9 mm to (91.8, 129.5), turned to 180 degrees
- moved TP2 25.6 mm to (87.5, 143.5)
- moved R9 23.9 mm to (90.0, 121.5), turned to 0 degrees
- moved TP3 22.6 mm to (94.0, 118.0)
- moved R8 21.6 mm to (89.0, 125.0)
- moved C4 20.8 mm to (93.5, 121.5)
- moved R14 20.5 mm to (111.5, 125.0)
- moved TP11 17.6 mm to (120.0, 131.5)
- moved C3 15.7 mm to (102.5, 124.5), turned to 270 degrees
- moved C6 15.6 mm to (111.0, 139.5), turned to 90 degrees
- moved TP6 14.8 mm to (87.5, 121.5), turned to 270 degrees
- moved C2 13.0 mm to (90.0, 136.0), turned to 0 degrees
- moved J3 12.4 mm to (120.0, 137.0), turned to 90 degrees
- moved C7 10.4 mm to (106.5, 129.0), turned to 180 degrees
- moved R7 10.1 mm to (96.5, 138.5)
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Connections:
- C2 pad 1: VCC -> Net-(C2-Pad1)
- C2 pad 2: GND -> Net-(C2-Pad2)
- C3 pad 1: GND -> VCC
- C3 pad 2: VCC -> GND
- C4 pad 1: Net-(C4-Pad1) -> GND
- C4 pad 2: Net-(C4-Pad2) -> VCC
- C6 pad 1: 3v3 -> Net-(C6-Pad1)
- C7 pad 1: GND -> 3v3
- C7 pad 2: 12v -> GND
- C8 pad 1: Net-(C8-Pad1) -> GND
- C8 pad 2: GND -> 12v
- J3 pad 1: Net-(J3-Pad1) -> GND
- J3 pad 2: Net-(J3-Pad2) -> Net-(C10-Pad2)
- Q1 pad 2: Net-(C4-Pad1) -> Net-(C2-Pad1)
- R10 pad 2: Net-(C8-Pad1) -> Net-(C6-Pad1)
- R12 pad 2: Net-(J3-Pad3) -> Net-(C10-Pad2)
- R13 pad 1: 3v3 -> Net-(C10-Pad2)
- R13 pad 2: Net-(C10-Pad2) -> GND
- R14 pad 1: Net-(C10-Pad2) -> Net-(R14-Pad1)
- R14 pad 2: GND -> 3v3
- R15 pad 1: 3v3 -> Net-(R14-Pad1)
- R15 pad 2: /SCL -> Net-(J3-Pad3)
- R16 pad 1: 3v3 -> GND
- R16 pad 2: /SDA -> Net-(R15-Pad3)
- R3 pad 1: Net-(C4-Pad1) -> Net-(C2-Pad1)
- R4 pad 2: Net-(C4-Pad2) -> Net-(C2-Pad2)
- R5 pad 1: Net-(C4-Pad2) -> Net-(C2-Pad2)
- R6 pad 1: 12v -> Net-(R6-Pad1)
- R7 pad 1: Net-(R6-Pad2) -> Net-(R6-Pad1)
- R7 pad 2: GND -> Net-(C5-Pad1)
- R8 pad 1: Net-(R8-Pad1) -> 12v
- R9 pad 1: Net-(R8-Pad1) -> Net-(R8-Pad2)
- R9 pad 2: Net-(C5-Pad1) -> GND
- TP2 pad 1: VCC -> Net-(C2-Pad1)
- TP3 pad 1: Net-(C4-Pad1) -> VCC
- TP4 pad 1: Net-(C4-Pad2) -> Net-(C2-Pad2)
- TP6 pad 1: Net-(R6-Pad2) -> Net-(R8-Pad2)
- TP8 pad 1: Net-(R8-Pad2) -> Net-(R6-Pad2)
- U1 pad 5: Net-(R6-Pad2) -> Net-(R8-Pad2)
- U2 pad 1: Net-(R8-Pad2) -> Net-(R6-Pad2)
- U2 pad 2: Net-(R8-Pad1) -> Net-(R6-Pad1)
- U2 pad 3: Net-(C4-Pad2) -> Net-(C2-Pad2)
- U2 pad 5: Net-(R8-Pad2) -> Net-(R6-Pad2)
Routing:
- net Net-(C2-Pad2): track 0.00 -> 21.5 mm
- net Net-(C4-Pad2): track 20.6 -> 0.00 mm
- net GND: track 18.8 -> 35.5 mm, vias 12 -> 16
- net Net-(C2-Pad1): track 0.00 -> 12.5 mm
- net Net-(C10-Pad2): track 8.34 -> 19.7 mm
- net Net-(C4-Pad1): track 9.52 -> 0.00 mm
- net Net-(R8-Pad2): track 16.5 -> 8.06 mm
- net 3v3: track 14.4 -> 22.5 mm
- net VCC: track 61.3 -> 53.9 mm
- net Net-(R8-Pad1): track 6.93 -> 0.00 mm
- net Net-(R6-Pad1): track 0.00 -> 6.93 mm
- net Net-(R6-Pad2): track 8.86 -> 15.5 mm
- net Net-(J3-Pad1): track 6.18 -> 0.00 mm
- net Net-(R14-Pad1): track 0.00 -> 3.45 mm
- net 12v: track 49.3 -> 46.2 mm
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Other:
- board size 42 x 36 mm -> 42 x 29.5 mm
- board text added: "G Brooks 2019"
- board text added: "TP10"
- board text added: "TP11"
- board text added: "TP2"
- board text added: "TP3"
- board text added: "TP4"
- board text added: "TP5"
- board text added: "TP8"
- board text added: "TP9"
- board text removed: "E"
- board text removed: "M"
- board text removed: "SCL"
- board text removed: "SDA"
- board text removed: "TP12"
- board text removed: "TPX"
- board text removed: "TPXX"
- board text removed: "Vin TPXX"

Commit message: Finish first revision of PCB
Parts:
- moved C10 0.25 mm to (110.0, 137.0)
Routing:
- net VCC: track 53.9 -> 56.2 mm

Commit message: Add gerbers
Routing:
- net GND: track 35.5 -> 39.5 mm
Changed lines of the file:
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@@
     (thickness 1.6)
     (drawings 25)
-    (tracks 259)
+    (tracks 263)
     (zones 0)
     (modules 46)
@@
     (visible_elements FFFFFF7F)
     (pcbplotparams
-      (layerselection 0x010fc_ffffffff)
+      (layerselection 0x010c0_ffffffff)
       (usegerberextensions false)
       (usegerberattributes false)
@@
       (outputformat 1)
       (mirror false)
-      (drillshape 1)
+      (drillshape 0)
       (scaleselection 1)
-      (outputdirectory ""))
+      (outputdirectory "gerbers/"))
   )
   (net 0 "")
@@
   (segment (start 116.3 131.5) (end 116.3 130.2) (width 0.5) (layer F.Cu) (net 2) (status 10))
   (segment (start 116.3 130.2) (end 117 129.5) (width 0.5) (layer F.Cu) (net 2))
+  (segment (start 84.6 118) (end 85.549999 118.950001) (width 0.5) (layer B.Cu) (net 2))
+  (segment (start 85.549999 118.950001) (end 86 119.400002) (width 0.5) (layer B.Cu) (net 2))
+  (segment (start 84.6 118) (end 83.5 119.1) (width 0.5) (layer B.Cu) (net 2))
+  (segment (start 83.5 119.1) (end 83.5 119.5) (width 0.5) (layer B.Cu) (net 2))
   (segment (start 99.725 123.275) (end 99.75 123.25) (width 0.5) (layer F.Cu) (net 3) (status 30))
   (segment (start 99.725 124.075) (end 99.725 123.275) (width 0.5) (layer F.Cu) (net 3) (status 30))
@@
     (polygon
       (pts
-        (xy 80 116) (xy 80 145.5) (xy 122 145.5) (xy 122 116)
+        (xy 88.5 116) (xy 88.5 117.5) (xy 80 117.5) (xy 80 145.5) (xy 122 145.5)
+        (xy 122 116)
       )
     )
