File: hardware-rng/hardware-rng.kicad_pcb (KiCad board)
At the start: 2 copper layers, 42 x 29.5 mm, 46 parts, among them IC1 MCP1700, J1 MICROUSB, J2 CONN_01x03, J3 CONN_01x03, Q1 2N4401, U1 ST8R00, U2 LT1215CS8#PBF

Commit message: Replace the word 'zener', since the circuit uses avalanche, rather than zener breakdown
Parts:
- L1: footprint zener-rng:WURTH_IND_3.8_3.8_1.65 -> hardware-rng:WURTH_IND_3.8_3.8_1.65
- Q1: footprint zener-rng:TO-92 -> hardware-rng:TO-92
- R15: footprint zener-rng:3266W_trimpot -> hardware-rng:3266W_trimpot
- U1: footprint zener-rng:DFN-8-ST -> hardware-rng:DFN-8-ST
Changed lines of the file:
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@@
   (page A4)
   (title_block
-    (title Zener-RNG)
+    (title Hardware-RNG)
     (date 2019-03-09)
     (rev 1.0)
@@
     )
   )
-  (module zener-rng:WURTH_IND_3.8_3.8_1.65 (layer F.Cu)
+  (module hardware-rng:WURTH_IND_3.8_3.8_1.65 (layer F.Cu)
     (at 98 125)
     (fp_text reference L1 (at 0 3.5) (layer F.Fab)
@@
       (net 15 "Net-(L1-Pad2)"))
   )
-  (module zener-rng:TO-92 (layer F.Cu)
+  (module hardware-rng:TO-92 (layer F.Cu)
     (at 89 138.5 270)
     (descr "TO-92 leads molded, narrow, drill 0.75mm (see NXP sot054_po.pdf)")
@@
       (net 14 "Net-(J3-Pad3)"))
   )
-  (module zener-rng:DFN-8-ST (layer F.Cu)
+  (module hardware-rng:DFN-8-ST (layer F.Cu)
     (at 92.5 125.5 180)
     (fp_text reference U1 (at 0 -3.3 180) (layer F.Fab)
@@
     )
   )
-  (module zener-rng:3266W_trimpot (layer F.Cu)
+  (module hardware-rng:3266W_trimpot (layer F.Cu)
     (at 116 126.2 270)
     (fp_text reference R15 (at 0 3.3 270) (layer F.Fab)
