File: hardware-rng/hardware-rng.sch (KiCad schematic (older format))
At the start: 46 parts, among them IC1 MCP1700, J1 MICROUSB, J2 CONN_01x03, J3 CONN_01x03, Q1 2N4401, U1 ST8R00, U2 LT1215CS8#PBF

Commit message: Replace the word 'zener', since the circuit uses avalanche, rather than zener breakdown
Parts:
- L1: footprint zener-rng:WURTH_IND_3.8_3.8_1.65 -> hardware-rng:WURTH_IND_3.8_3.8_1.65
- Q1: footprint zener-rng:TO-92 -> hardware-rng:TO-92
- R15: footprint zener-rng:3266W_trimpot -> hardware-rng:3266W_trimpot
- U1: footprint zener-rng:DFN-8-ST -> hardware-rng:DFN-8-ST
Other:
- note added: "hardware"
- note removed: "zener"
Changed lines of the file:
@@
 EESchema Schematic File Version 4
-LIBS:zener-rng-cache
+LIBS:hardware-rng-cache
 EELAYER 26 0
 EELAYER END
@@
 encoding utf-8
 Sheet 1 1
-Title "Zener-RNG"
+Title "Hardware-RNG"
 Date "2019-03-08"
 Rev "1.0"
@@
 $EndComp
 Text Notes 2550 2350 0    50   ~ 0
-zener
+hardware
 $Comp
 L agg-kicad:R R1
@@
 F 0 "Q1" H 3638 2654 50  0000 L CNN
 F 1 "2N4401" H 3638 2745 50  0000 L CNN
-F 2 "zener-rng:TO-92" H 3530 2620 50  0001 C CNN
+F 2 "hardware-rng:TO-92" H 3530 2620 50  0001 C CNN
 F 3 "http://www.farnell.com/datasheets/1702446.pdf" H 3630 2720 50  0001 C CNN
 F 4 "1574373" H 3500 2700 50  0001 C CNN "Farnell"
@@
 F 0 "L1" H 3000 6228 50  0000 C CNN
 F 1 "4.7uH" H 3000 6137 50  0000 C CNN
-F 2 "zener-rng:WURTH_IND_3.8_3.8_1.65" H 2950 6050 50  0001 C CNN
+F 2 "hardware-rng:WURTH_IND_3.8_3.8_1.65" H 2950 6050 50  0001 C CNN
 F 3 "http://www.farnell.com/datasheets/1910986.pdf" H 2950 6050 50  0001 C CNN
 F 4 "1635834" H 2950 6050 50  0001 C CNN "Farnell"
@@
 F 0 "U1" H 2510 6796 50  0000 R CNN
 F 1 "ST8R00" H 2510 6705 50  0000 R CNN
-F 2 "zener-rng:DFN-8-ST" H 3000 5600 50  0001 C CNN
+F 2 "hardware-rng:DFN-8-ST" H 3000 5600 50  0001 C CNN
 F 3 "http://www.farnell.com/datasheets/2581721.pdf" H 3000 5700 50  0001 C CNN
 F 4 "2849799" H 3000 5500 50  0001 C CNN "Farnell"
@@
 F 0 "R15" V 7604 1938 50  0000 L CNN
 F 1 "1k potentiometer" V 7695 1938 50  0000 L CNN
-F 2 "zener-rng:3266W_trimpot" H 7650 1850 50  0001 C CNN
+F 2 "hardware-rng:3266W_trimpot" H 7650 1850 50  0001 C CNN
 F 3 "http://www.farnell.com/datasheets/2061259.pdf" H 7650 1850 50  0001 C CNN
 F 4 "9352643" H 7650 1850 50  0001 C CNN "Farnell"

Commit message: Remove leftover comment from schematic
Other:
- note removed: "hardware"
Changed lines of the file:
@@
 	0    1    1    0
 $EndComp
-Text Notes 2550 2350 0    50   ~ 0
-hardware
 $Comp
 L agg-kicad:R R1
